File: src/PCB/feeder-slot/feederSlot.kicad_sch (KiCad schematic)
At the start: 6 parts, among them J2 Conn_01x05_Female, J3 Conn_01x04_Pin, U1 DS28E07

Commit message: cleanup
Parts:
- R1: LCSC C61683 -> C114245
- R2: LCSC C61683 -> (none)
Changed lines of the file:
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@@
 			)
 		)
-		(property "LCSC" "C61683"
+		(property "LCSC" "C114245"
 			(at 97.79 134.62 0)
 			(effects
@@
 			)
 		)
-		(property "LCSC" "C61683"
-			(at 168.91 133.35 0)
-			(effects
+		(property "LCSC" ""
+			(at 168.91 133.35 0)
+			(effects
