File: src/PCB/power-breakout/power-breakout.kicad_pcb (KiCad board)
At the start: 2 copper layers, 48 x 50 mm, 29 parts, among them J1 COMBO_POWER_JACK, J2 Conn_01x04_Pin, U1 FDS4435BZ, U2 FDS4435BZ

Commit message: cleanup
Other:
- board text added: "Opulo Feeder Loading Station Power Board REV00 - 629777d"
- board text removed: "Opulo Feeder Loading Station Power Board REV00"
